File: board/KiCad/ice40.sch (KiCad schematic (older format))
At the start: 4 parts, among them U1 iCE40_1K4K_TQ144

Commit message: DIQ1 Bus added
Connections:
- net DIQ1_D0: now reaches U1.73 (IOR_48_109)
- net DIQ1_D1: now reaches U1.74 (IOR_49_110)
- net DIQ1_D2: now reaches U1.75 (IOR_50_111)
- net DIQ1_D3: now reaches U1.76 (IOR_51_112)
- net DIQ1_D4: now reaches U1.78 (IOR_52_114)
- net DIQ1_D5: now reaches U1.79 (IOR_53_115)
- net DIQ1_D6: now reaches U1.80 (IOR_54_116)
- net DIQ1_D7: now reaches U1.81 (IOR_55_117)
- net DIQ1_D8: now reaches U1.87 (IOR_56_136)
- net DIQ1_D9: now reaches U1.88 (IOR_57_137)
- net DIQ1_D10: now reaches U1.90 (IOR_58_138)
- net DIQ1_D11: now reaches U1.91 (IOR_59_139)
Changed lines of the file:
@@
 	2250 1250 2250 1350
 Connection ~ 1950 1250
+Wire Bus Line
+	5300 800  5300 2250
+Entry Bus Bus
+	5300 2250 5400 2350
+Text GLabel 5400 2350 2    60   Input ~ 0
+DIQ1
+Entry Wire Line
+	5200 950  5300 1050
+Entry Wire Line
+	5200 1050 5300 1150
+Entry Wire Line
+	5200 1150 5300 1250
+Entry Wire Line
+	5200 1250 5300 1350
+Entry Wire Line
+	5200 1350 5300 1450
+Entry Wire Line
+	5200 1450 5300 1550
+Entry Wire Line
+	5200 1550 5300 1650
+Entry Wire Line
+	5200 1650 5300 1750
+Entry Wire Line
+	5200 1750 5300 1850
+Entry Wire Line
+	5200 1850 5300 1950
+Entry Wire Line
+	5200 1950 5300 2050
+Entry Wire Line
+	5200 2050 5300 2150
+Wire Wire Line
+	4700 950  5200 950
+Wire Wire Line
+	4700 1050 5200 1050
+Wire Wire Line
+	4700 1150 5200 1150
+Wire Wire Line
+	4700 1250 5200 1250
+Wire Wire Line
+	4700 1350 5200 1350
+Wire Wire Line
+	4700 1450 5200 1450
+Wire Wire Line
+	4700 1550 5200 1550
+Wire Wire Line
+	4700 1650 5200 1650
+Wire Wire Line
+	4700 1750 5200 1750
+Wire Wire Line
+	4700 1850 5200 1850
+Wire Wire Line
+	4700 1950 5200 1950
+Wire Wire Line
+	4700 2050 5200 2050
+Text Label 4750 950  0    60   ~ 0
+DIQ1_D0
+Text Label 4750 1050 0    60   ~ 0
+DIQ1_D1
+Text Label 4750 1150 0    60   ~ 0
+DIQ1_D2
+Text Label 4750 1250 0    60   ~ 0
+DIQ1_D3
+Text Label 4750 1350 0    60   ~ 0
+DIQ1_D4
+Text Label 4750 1450 0    60   ~ 0
+DIQ1_D5
+Text Label 4750 1550 0    60   ~ 0
+DIQ1_D6
+Text Label 4750 1650 0    60   ~ 0
+DIQ1_D7
+Text Label 4750 1750 0    60   ~ 0
+DIQ1_D8
+Text Label 4750 1850 0    60   ~ 0
+DIQ1_D9
+Text Label 4750 1950 0    60   ~ 0
+DIQ1_D10
+Text Label 4750 2050 0    60   ~ 0
+DIQ1_D11
 $EndSCHEMATC

Commit message: DIQ2 Bus added
Connections:
- net DIQ2_D6: now reaches U1.101 (IOR_67_160)
- net DIQ2_D7: now reaches U1.102 (IOR_68_161)
- net DIQ2_D8: now reaches U1.104 (IOR_69_164)
- net DIQ2_D9: now reaches U1.105 (IOR_70_165)
- net DIQ2_D10: now reaches U1.106 (IOR_71_166)
- net DIQ2_D11: now reaches U1.107 (IOR_72_167)
- net DIQ2_D0: now reaches U1.94 (IOR_61_141)
- net DIQ2_D1: now reaches U1.95 (IOR_62_144)
- net DIQ2_D2: now reaches U1.96 (IOR_63_146)
- net DIQ2_D3: now reaches U1.97 (IOR_64_147)
- net DIQ2_D4: now reaches U1.98 (IOR_65_148)
- net DIQ2_D5: now reaches U1.99 (IOR_66_152)
Changed lines of the file:
@@
 Text Label 4750 2050 0    60   ~ 0
 DIQ1_D11
+Wire Wire Line
+	4700 2350 5200 2350
+Wire Wire Line
+	4700 2450 5200 2450
+Wire Wire Line
+	4700 2550 5200 2550
+Wire Wire Line
+	4700 2650 5200 2650
+Wire Wire Line
+	4700 2750 5200 2750
+Wire Wire Line
+	4700 2850 5200 2850
+Wire Wire Line
+	4700 2950 5200 2950
+Wire Wire Line
+	4700 3050 5200 3050
+Wire Wire Line
+	4700 3150 5200 3150
+Wire Wire Line
+	4700 3250 5200 3250
+Wire Wire Line
+	4700 3350 5200 3350
+Wire Wire Line
+	4700 2250 5200 2250
+Entry Wire Line
+	5200 2250 5300 2350
+Entry Wire Line
+	5200 2350 5300 2450
+Entry Wire Line
+	5200 2450 5300 2550
+Entry Wire Line
+	5200 2550 5300 2650
+Entry Wire Line
+	5200 2650 5300 2750
+Entry Wire Line
+	5200 2750 5300 2850
+Entry Wire Line
+	5200 2850 5300 2950
+Entry Wire Line
+	5200 2950 5300 3050
+Entry Wire Line
+	5200 3050 5300 3150
+Entry Wire Line
+	5200 3150 5300 3250
+Entry Wire Line
+	5200 3250 5300 3350
+Entry Wire Line
+	5200 3350 5300 3450
+Wire Bus Line
+	5300 2350 5300 3500
+Entry Bus Bus
+	5300 3500 5400 3600
+Text GLabel 5400 3600 2    60   Input ~ 0
+DIQ2
+Text Label 4750 2250 0    60   ~ 0
+DIQ2_D0
+Text Label 4750 2350 0    60   ~ 0
+DIQ2_D1
+Text Label 4750 2450 0    60   ~ 0
+DIQ2_D2
+Text Label 4750 2550 0    60   ~ 0
+DIQ2_D3
+Text Label 4750 2650 0    60   ~ 0
+DIQ2_D4
+Text Label 4750 2750 0    60   ~ 0
+DIQ2_D5
+Text Label 4750 2850 0    60   ~ 0
+DIQ2_D6
+Text Label 4750 2950 0    60   ~ 0
+DIQ2_D7
+Text Label 4750 3050 0    60   ~ 0
+DIQ2_D8
+Text Label 4750 3150 0    60   ~ 0
+DIQ2_D9
+Text Label 4750 3250 0    60   ~ 0
+DIQ2_D10
+Text Label 4750 3350 0    60   ~ 0
+DIQ2_D11
 $EndSCHEMATC

Commit message: control signals added
Connections:
- net at U1.123 (VCCIO_0): now also U1.133 (VCCIO_0)
- net ICE_CLK_IN: now reaches U1.21 (GBIN6)
- net at U1.46 (VCCIO_2): now also U1.57 (VCCIO_2)
- net RXEN: now reaches U1.112 (IOT_73_169)
- net TXEN: now reaches U1.113 (IOT_74_170)
- net DIQ1_SEL: now reaches U1.114 (IOT_75_171)
- net DIQ2_SEL: now reaches U1.115 (IOT_76_172)
- net FCLK1: now reaches U1.116 (IOT_77_173)
- net FCLK2: now reaches U1.117 (IOT_78_174)
- net RFDIO_RESET: now reaches U1.118 (IOT_79_177)
- net RFDIO_GPIO0: now reaches U1.119 (IOT_80_178)
- net RFDIO_GPIO1: now reaches U1.120 (IOT_81_179)
- net RFDIO_GPIO2: now reaches U1.121 (IOT_82_181)
- net RFDIO_SPI_MOSI: now reaches U1.122 (IOT_83_190)
- net RFDIO_SPI_MISO: now reaches U1.128 (IOT_84_197)
- net RFDIO_SPI_CLK: now reaches U1.129 (IOT_85_198)
- net RFDIO_SPI_EN: now reaches U1.134 (IOT_87_212)
- net RFDIO_REF_CLK_IN: now reaches U1.135 (IOT_88_213)
Changed lines of the file:
@@
 Text Label 4750 3350 0    60   ~ 0
 DIQ2_D11
+Wire Wire Line
+	1700 3050 1850 3050
+Wire Wire Line
+	1850 3050 1850 3150
+Wire Wire Line
+	1850 3150 1700 3150
+Wire Wire Line
+	1700 3450 1850 3450
+Wire Wire Line
+	1850 3450 1850 3550
+Wire Wire Line
+	1850 3550 1700 3550
+Wire Wire Line
+	1700 4800 2050 4800
+Wire Wire Line
+	1700 4900 2050 4900
+Text GLabel 2050 4800 2    60   Input ~ 0
+RXEN
+Text GLabel 2050 4900 2    60   Input ~ 0
+TXEN
+Wire Wire Line
+	1700 5000 2050 5000
+Wire Wire Line
+	1700 5100 2050 5100
+Text GLabel 2050 5000 2    60   Input ~ 0
+DIQ1_SEL
+Text GLabel 2050 5100 2    60   Input ~ 0
+DIQ2_SEL
+Wire Wire Line
+	1700 5200 2050 5200
+Wire Wire Line
+	1700 5300 2050 5300
+Text GLabel 2050 5200 2    60   Input ~ 0
+FCLK1
+Text GLabel 2050 5300 2    60   Input ~ 0
+FCLK2
+Wire Wire Line
+	1700 1150 1950 1150
+Text GLabel 1950 1150 2    60   Input ~ 0
+ICE_CLK_IN
+Wire Wire Line
+	1700 5400 2050 5400
+Wire Wire Line
+	1700 5500 2050 5500
+Wire Wire Line
+	1700 5600 2050 5600
+Wire Wire Line
+	1700 5700 2050 5700
+Text GLabel 2050 5400 2    60   Input ~ 0
+RFDIO_RESET
+Text GLabel 2050 5500 2    60   Input ~ 0
+RFDIO_GPIO0
+Text GLabel 2050 5600 2    60   Input ~ 0
+RFDIO_GPIO1
+Text GLabel 2050 5700 2    60   Input ~ 0
+RFDIO_GPIO2
+Text GLabel 2050 5800 2    60   Input ~ 0
+RFDIO_SPI_MOSI
+Text GLabel 2050 5900 2    60   Input ~ 0
+RFDIO_SPI_MISO
+Text GLabel 2050 6000 2    60   Input ~ 0
+RFDIO_SPI_CLK
+Text GLabel 2050 6100 2    60   Input ~ 0
+RFDIO_SPI_EN
+Wire Wire Line
+	1700 5800 2050 5800
+Wire Wire Line
+	1700 5900 2050 5900
+Wire Wire Line
+	1700 6000 2050 6000
+Wire Wire Line
+	1700 6100 2050 6100
+Wire Wire Line
+	1700 6200 2050 6200
+Text GLabel 2050 6200 2    60   Input ~ 0
+RFDIO_REF_CLK_IN
 $EndSCHEMATC
