File: board/KiCad/ice40.sch (KiCad schematic (older format))
At the start: 4 parts, among them U1 iCE40_1K4K_TQ144

Commit message: spi & reset
Parts:
- added R? (x3): 10K, symbol R
Connections:
- net +3V3: now also U1.123 (VCCIO_0), U1.133 (VCCIO_0), U1.46 (VCCIO_2), U1.57 (VCCIO_2), U1.72 (VCC_SPI), R?.1, R?.1
- net GND: now also R?.2
- net ICE_CDONE: now reaches U1.65 (CDONE)
- net ICE_CDONE: now also R?.2
- net ICE_CRESET_B: now reaches U1.66 (CRESET_B)
- net ICE_CRESET_B: now also R?.1, R?.2
- net ICE_SDO: now reaches U1.67 (SDO)
- net ICE_SDI: now reaches U1.68 (SDI)
- net ICE_SCK: now reaches U1.70 (SCK)
- net ICE_SS: now reaches U1.71 (SS)
Changed lines of the file:
@@
 Text GLabel 8950 2400 2    60   Input ~ 0
 PIO7
-$Comp
-L +3V3 #PWR6
-U 1 1 56A62583
-P 2050 3700
-F 0 "#PWR6" H 2050 3550 50  0001 C CNN
-F 1 "+3V3" H 2068 3874 50  0000 C CNN
-F 2 "" H 2050 3700 50  0000 C CNN
-F 3 "" H 2050 3700 50  0000 C CNN
-	1    2050 3700
-	1    0    0    -1
-$EndComp
 Text GLabel 4250 7400 0    60   Input ~ 0
 3V3_PMOD
@@
 L +1V2 #PWR7
 U 1 1 56ABC35C
-P 2100 2650
-F 0 "#PWR7" H 2100 2500 50  0001 C CNN
-F 1 "+1V2" H 2100 2790 50  0000 C CNN
-F 2 "" H 2100 2650 60  0000 C CNN
-F 3 "" H 2100 2650 60  0000 C CNN
-	1    2100 2650
+P 2300 2650
+F 0 "#PWR7" H 2300 2500 50  0001 C CNN
+F 1 "+1V2" H 2300 2790 50  0000 C CNN
+F 2 "" H 2300 2650 60  0000 C CNN
+F 3 "" H 2300 2650 60  0000 C CNN
+	1    2300 2650
 	1    0    0    -1
 $EndComp
@@
 	8250 2300 8600 2300
 Wire Wire Line
-	1700 3750 1850 3750
-Wire Wire Line
-	1850 3750 1850 3650
+	1850 3750 1700 3750
+Wire Wire Line
+	1850 3050 1850 3750
 Wire Wire Line
 	1850 3650 1700 3650
 Wire Wire Line
-	1850 3700 2050 3700
-Connection ~ 1850 3700
-Wire Wire Line
 	4250 7400 4900 7400
 Wire Wire Line
@@
 	5100 7650 5100 7600
 Wire Wire Line
-	1700 2650 2100 2650
+	1700 2650 2300 2650
 Wire Wire Line
 	1850 2650 1850 2950
@@
 Wire Wire Line
 	1700 3250 1850 3250
-Wire Wire Line
-	1850 3250 1850 3350
 Wire Wire Line
 	1850 3350 1700 3350
@@
 	1700 3050 1850 3050
 Wire Wire Line
-	1850 3050 1850 3150
-Wire Wire Line
 	1850 3150 1700 3150
 Wire Wire Line
-	1700 3450 1850 3450
-Wire Wire Line
-	1850 3450 1850 3550
+	1850 3450 1700 3450
 Wire Wire Line
 	1850 3550 1700 3550
@@
 Text GLabel 2050 6200 2    60   Input ~ 0
 RFDIO_REF_CLK_IN
+Text GLabel 1700 1050 2    60   Input ~ 0
+ICE_CRESET_B
+Text GLabel 1700 950  2    60   Input ~ 0
+ICE_CDONE
+Text GLabel 1700 2250 2    60   Input ~ 0
+ICE_SCK
+Text GLabel 1700 2350 2    60   Input ~ 0
+ICE_SDI
+Text GLabel 1700 2450 2    60   Input ~ 0
+ICE_SDO
+Text GLabel 1700 2550 2    60   Input ~ 0
+ICE_SS
+$Comp
+L +3V3 #PWR?
+U 1 1 56BB434D
+P 2250 4100
+F 0 "#PWR?" H 2250 3950 50  0001 C CNN
+F 1 "+3V3" H 2268 4274 50  0000 C CNN
+F 2 "" H 2250 4100 50  0000 C CNN
+F 3 "" H 2250 4100 50  0000 C CNN
+	1    2250 4100
+	1    0    0    -1
+$EndComp
+Wire Wire Line
+	1700 3950 2100 3950
+Wire Wire Line
+	2100 3950 2100 4100
+Wire Wire Line
+	2100 4100 2250 4100
+Connection ~ 1850 3250
+Connection ~ 1850 3150
+Connection ~ 1850 3450
+Connection ~ 1850 3350
+Connection ~ 1850 3650
+Connection ~ 1850 3550
+Text GLabel 7100 4950 0    60   Input ~ 0
+ICE_CDONE
+$Comp
+L R R?
+U 1 1 56BB4D04
+P 7350 4600
+F 0 "R?" V 7430 4600 50  0000 C CNN
+F 1 "10K" V 7350 4600 50  0000 C CNN
+F 2 "" V 7280 4600 30  0000 C CNN
+F 3 "" H 7350 4600 30  0000 C CNN
+	1    7350 4600
+	1    0    0    -1
+$EndComp
+Wire Wire Line
+	7100 4950 7350 4950
+Wire Wire Line
+	7350 4950 7350 4750
+$Comp
+L +3V3 #PWR?
+U 1 1 56BB5247
+P 7350 4350
+F 0 "#PWR?" H 7350 4200 50  0001 C CNN
+F 1 "+3V3" H 7368 4524 50  0000 C CNN
+F 2 "" H 7350 4350 50  0000 C CNN
+F 3 "" H 7350 4350 50  0000 C CNN
+	1    7350 4350
+	1    0    0    -1
+$EndComp
+Wire Wire Line
+	7350 4450 7350 4350
+Text GLabel 8450 4950 0    60   Input ~ 0
+ICE_CRESET_B
+$Comp
+L R R?
+U 1 1 56BB5708
+P 8750 4600
+F 0 "R?" V 8830 4600 50  0000 C CNN
+F 1 "10K" V 8750 4600 50  0000 C CNN
+F 2 "" V 8680 4600 30  0000 C CNN
+F 3 "" H 8750 4600 30  0000 C CNN
+	1    8750 4600
+	1    0    0    -1
+$EndComp
+$Comp
+L +3V3 #PWR?
+U 1 1 56BB576D
+P 8750 4350
+F 0 "#PWR?" H 8750 4200 50  0001 C CNN
+F 1 "+3V3" H 8768 4524 50  0000 C CNN
+F 2 "" H 8750 4350 50  0000 C CNN
+F 3 "" H 8750 4350 50  0000 C CNN
+	1    8750 4350
+	1    0    0    -1
+$EndComp
+Wire Wire Line
+	8450 4950 8750 4950
+Wire Wire Line
+	8750 4750 8750 5150
+Wire Wire Line
+	8750 4450 8750 4350
+$Comp
+L R R?
+U 1 1 56BB5AAD
+P 8750 5300
+F 0 "R?" V 8830 5300 50  0000 C CNN
+F 1 "10K" V 8750 5300 50  0000 C CNN
+F 2 "" V 8680 5300 30  0000 C CNN
+F 3 "" H 8750 5300 30  0000 C CNN
+	1    8750 5300
+	1    0    0    -1
+$EndComp
+$Comp
+L GND #PWR?
+U 1 1 56BB5D2F
+P 8750 5650
+F 0 "#PWR?" H 8750 5400 50  0001 C CNN
+F 1 "GND" H 8750 5500 50  0000 C CNN
+F 2 "" H 8750 5650 60  0000 C CNN
+F 3 "" H 8750 5650 60  0000 C CNN
+	1    8750 5650
+	1    0    0    -1
+$EndComp
+Connection ~ 8750 4950
+Wire Wire Line
+	8750 5650 8750 5450
 $EndSCHEMATC

Commit message: SPI & Osci
Parts:
- added C? (x2): 10µF, symbol C
- added C? (x2): 1µF, symbol C
- added C? (x2): 0.1µF, symbol C
- added C? (x2): 0.01µF, symbol C
- added D?: LED, symbol LED
- added R?: 10, symbol R
- R?: value 10K -> 0
Connections:
- net +1V2: now also C?.1, C?.1, C?.1, C?.1
- net +3V3: now also C?.1, C?.1, C?.1, C?.1
- net GND: now also C?.2, C?.2, C?.2, C?.2, C?.2, C?.2, C?.2, C?.2, D?.1 (K)
- net ICE_CDONE: now also R?.1
- new net: D?.2 (A), R?.2
Other:
- moved on the sheet: R?
Changed lines of the file:
@@
 $Descr A4 11693 8268
 encoding utf-8
-Sheet 3 5
+Sheet 3 6
 Title ""
 Date ""
@@
 	3350 3850 3450 3850
 Wire Wire Line
-	1700 2050 1950 2050
-Wire Wire Line
-	1950 2050 1950 1250
+	1950 2050 1700 2050
+Wire Wire Line
+	1950 1250 1950 2050
 Wire Wire Line
 	1700 1250 2250 1250
@@
 Connection ~ 1850 3650
 Connection ~ 1850 3550
-Text GLabel 7100 4950 0    60   Input ~ 0
+Text GLabel 6650 3750 0    60   Input ~ 0
 ICE_CDONE
 $Comp
 L R R?
 U 1 1 56BB4D04
-P 7350 4600
-F 0 "R?" V 7430 4600 50  0000 C CNN
-F 1 "10K" V 7350 4600 50  0000 C CNN
-F 2 "" V 7280 4600 30  0000 C CNN
-F 3 "" H 7350 4600 30  0000 C CNN
-	1    7350 4600
-	1    0    0    -1
-$EndComp
-Wire Wire Line
-	7100 4950 7350 4950
-Wire Wire Line
-	7350 4950 7350 4750
+P 6900 3400
+F 0 "R?" V 6980 3400 50  0000 C CNN
+F 1 "10K" V 6900 3400 50  0000 C CNN
+F 2 "" V 6830 3400 30  0000 C CNN
+F 3 "" H 6900 3400 30  0000 C CNN
+	1    6900 3400
+	1    0    0    -1
+$EndComp
+Wire Wire Line
+	6650 3750 6900 3750
+Wire Wire Line
+	6900 3550 6900 3850
 $Comp
 L +3V3 #PWR?
 U 1 1 56BB5247
-P 7350 4350
-F 0 "#PWR?" H 7350 4200 50  0001 C CNN
-F 1 "+3V3" H 7368 4524 50  0000 C CNN
-F 2 "" H 7350 4350 50  0000 C CNN
-F 3 "" H 7350 4350 50  0000 C CNN
-	1    7350 4350
-	1    0    0    -1
-$EndComp
-Wire Wire Line
-	7350 4450 7350 4350
+P 6900 3150
+F 0 "#PWR?" H 6900 3000 50  0001 C CNN
+F 1 "+3V3" H 6918 3324 50  0000 C CNN
+F 2 "" H 6900 3150 50  0000 C CNN
+F 3 "" H 6900 3150 50  0000 C CNN
+	1    6900 3150
+	1    0    0    -1
+$EndComp
+Wire Wire Line
+	6900 3250 6900 3150
 Text GLabel 8450 4950 0    60   Input ~ 0
 ICE_CRESET_B
@@
 P 8750 5300
 F 0 "R?" V 8830 5300 50  0000 C CNN
-F 1 "10K" V 8750 5300 50  0000 C CNN
+F 1 "0" V 8750 5300 50  0000 C CNN
 F 2 "" V 8680 5300 30  0000 C CNN
 F 3 "" H 8750 5300 30  0000 C CNN
@@
 Wire Wire Line
 	8750 5650 8750 5450
+$Comp
+L C C?
+U 1 1 56BB983C
+P 6450 5950
+F 0 "C?" H 6475 6050 50  0000 L CNN
+F 1 "10µF" H 6475 5850 50  0000 L CNN
+F 2 "" H 6488 5800 30  0001 C CNN
+F 3 "" H 6450 5950 60  0000 C CNN
+	1    6450 5950
+	1    0    0    -1
+$EndComp
+$Comp
+L C C?
+U 1 1 56BB98C5
+P 6800 5950
+F 0 "C?" H 6825 6050 50  0000 L CNN
+F 1 "1µF" H 6825 5850 50  0000 L CNN
+F 2 "" H 6838 5800 30  0001 C CNN
+F 3 "" H 6800 5950 60  0000 C CNN
+	1    6800 5950
+	1    0    0    -1
+$EndComp
+$Comp
+L C C?
+U 1 1 56BB9909
+P 7150 5950
+F 0 "C?" H 7175 6050 50  0000 L CNN
+F 1 "0.1µF" H 7175 5850 50  0000 L CNN
+F 2 "" H 7188 5800 30  0001 C CNN
+F 3 "" H 7150 5950 60  0000 C CNN
+	1    7150 5950
+	1    0    0    -1
+$EndComp
+$Comp
+L C C?
+U 1 1 56BB996E
+P 7500 5950
+F 0 "C?" H 7525 6050 50  0000 L CNN
+F 1 "0.01µF" H 7525 5850 50  0000 L CNN
+F 2 "" H 7538 5800 30  0001 C CNN
+F 3 "" H 7500 5950 60  0000 C CNN
+	1    7500 5950
+	1    0    0    -1
+$EndComp
+Wire Wire Line
+	6450 5800 7500 5800
+Connection ~ 6800 5800
+Connection ~ 7150 5800
+Wire Wire Line
+	6450 6100 7500 6100
+Connection ~ 6800 6100
+Connection ~ 7150 6100
+$Comp
+L GND #PWR?
+U 1 1 56BB9E95
+P 7150 6200
+F 0 "#PWR?" H 7150 5950 50  0001 C CNN
+F 1 "GND" H 7150 6050 50  0000 C CNN
+F 2 "" H 7150 6200 60  0000 C CNN
+F 3 "" H 7150 6200 60  0000 C CNN
+	1    7150 6200
+	1    0    0    -1
+$EndComp
+$Comp
+L +3V3 #PWR?
+U 1 1 56BB9ED0
+P 7150 5650
+F 0 "#PWR?" H 7150 5500 50  0001 C CNN
+F 1 "+3V3" H 7168 5824 50  0000 C CNN
+F 2 "" H 7150 5650 50  0000 C CNN
+F 3 "" H 7150 5650 50  0000 C CNN
+	1    7150 5650
+	1    0    0    -1
+$EndComp
+Wire Wire Line
+	7150 5650 7150 5800
+Wire Wire Line
+	7150 6100 7150 6200
+$Comp
+L C C?
+U 1 1 56BBA586
+P 4400 6500
+F 0 "C?" H 4425 6600 50  0000 L CNN
+F 1 "10µF" H 4425 6400 50  0000 L CNN
+F 2 "" H 4438 6350 30  0001 C CNN
+F 3 "" H 4400 6500 60  0000 C CNN
+	1    4400 6500
+	1    0    0    -1
+$EndComp
+$Comp
+L C C?
+U 1 1 56BBA58C
+P 4750 6500
+F 0 "C?" H 4775 6600 50  0000 L CNN
+F 1 "1µF" H 4775 6400 50  0000 L CNN
+F 2 "" H 4788 6350 30  0001 C CNN
+F 3 "" H 4750 6500 60  0000 C CNN
+	1    4750 6500
+	1    0    0    -1
+$EndComp
+$Comp
+L C C?
+U 1 1 56BBA592
+P 5100 6500
+F 0 "C?" H 5125 6600 50  0000 L CNN
+F 1 "0.1µF" H 5125 6400 50  0000 L CNN
+F 2 "" H 5138 6350 30  0001 C CNN
+F 3 "" H 5100 6500 60  0000 C CNN
+	1    5100 6500
+	1    0    0    -1
+$EndComp
+$Comp
+L C C?
+U 1 1 56BBA598
+P 5450 6500
+F 0 "C?" H 5475 6600 50  0000 L CNN
+F 1 "0.01µF" H 5475 6400 50  0000 L CNN
+F 2 "" H 5488 6350 30  0001 C CNN
+F 3 "" H 5450 6500 60  0000 C CNN
+	1    5450 6500
+	1    0    0    -1
+$EndComp
+Wire Wire Line
+	4400 6350 5450 6350
+Connection ~ 4750 6350
+Connection ~ 5100 6350
+Wire Wire Line
+	4400 6650 5450 6650
+Connection ~ 4750 6650
+Connection ~ 5100 6650
+$Comp
+L GND #PWR?
+U 1 1 56BBA5A4
+P 5100 6750
+F 0 "#PWR?" H 5100 6500 50  0001 C CNN
+F 1 "GND" H 5100 6600 50  0000 C CNN
+F 2 "" H 5100 6750 60  0000 C CNN
+F 3 "" H 5100 6750 60  0000 C CNN
+	1    5100 6750
+	1    0    0    -1
+$EndComp
+Wire Wire Line
+	5100 6200 5100 6350
+Wire Wire Line
+	5100 6650 5100 6750
+$Comp
+L +1V2 #PWR?
+U 1 1 56BBA638
+P 5100 6200
+F 0 "#PWR?" H 5100 6050 50  0001 C CNN
+F 1 "+1V2" H 5100 6340 50  0000 C CNN
+F 2 "" H 5100 6200 60  0000 C CNN
+F 3 "" H 5100 6200 60  0000 C CNN
+	1    5100 6200
+	1    0    0    -1
+$EndComp
+$Comp
+L R R?
+U 1 1 56BD2269
+P 6900 4000
+F 0 "R?" V 6980 4000 50  0000 C CNN
+F 1 "10" V 6900 4000 50  0000 C CNN
+F 2 "" V 6830 4000 30  0000 C CNN
+F 3 "" H 6900 4000 30  0000 C CNN
+	1    6900 4000
+	1    0    0    -1
+$EndComp
+$Comp
+L LED D?
+U 1 1 56BD2368
+P 6900 4450
+F 0 "D?" H 6900 4550 50  0000 C CNN
+F 1 "LED" H 6900 4350 50  0000 C CNN
+F 2 "" H 6900 4450 60  0000 C CNN
+F 3 "" H 6900 4450 60  0000 C CNN
+	1    6900 4450
+	0    -1   -1   0
+$EndComp
+$Comp
+L GND #PWR?
+U 1 1 56BD2668
+P 6900 4750
+F 0 "#PWR?" H 6900 4500 50  0001 C CNN
+F 1 "GND" H 6900 4600 50  0000 C CNN
+F 2 "" H 6900 4750 60  0000 C CNN
+F 3 "" H 6900 4750 60  0000 C CNN
+	1    6900 4750
+	1    0    0    -1
+$EndComp
+Connection ~ 6900 3750
+Wire Wire Line
+	6900 4250 6900 4150
+Wire Wire Line
+	6900 4750 6900 4650
 $EndSCHEMATC

Commit message: minor changes
Parts:
- removed R?: 0, symbol R
- added D?: Schottky 0520, symbol D_Schottky_Small
- added D? (x3): LED, symbol LED
- added R? (x3): 10, symbol R
- added SW?: ICE_RESET, SW_B3U-1000P, symbol SW_Tactile
Connections:
- net +3V3: now also D?.2 (A)
- net GND: now also D?.1 (K), D?.1 (K), D?.1 (K)
- net at U1.109 (VPP_FAST): now also D?.1 (K)
- net at U1.142 (IOT_94_220): now also R?.2
- net at U1.143 (IOT_95_221): now also R?.2
- net at U1.144 (IOT_96_222): now also R?.2
- new net: D?.2 (A), R?.1 (x3)
Other:
- note added: "ICE reset"
- note added: "LED prog. done"
- moved on the sheet: C?

Commit message: Finalize first draft
Parts:
- added C14, C15, C16, C17, C18, C19, C20, C21, C22, C23: 100n, Capacitors_SMD:C_0603_HandSoldering, symbol C_Small
- C1, C2: footprint (none) -> Capacitors_SMD:C_0603_HandSoldering
- C10, C11, C12, C13, C6, C7, C8, C9: renamed from C?; footprint (none) -> Capacitors_SMD:C_0603_HandSoldering
- D2: renamed from D?; footprint (none) -> pmod:SOD-123_Handsoldering
- D3, D4, D5, D6: renamed from D?; footprint (none) -> SMD_Packages:SMD-1206_Pol; symbol LED -> Led_Small
- R1: footprint (none) -> Resistors_SMD:R_0603_HandSoldering
- R12, R2, R3, R4, R7, R8: renamed from R?; footprint (none) -> Resistors_SMD:R_0603_HandSoldering
- SW1: renamed from SW?; footprint SW_B3U-1000P -> pmod:B3U-1000P_Handsoldering; Description SWITCH, TACTILE, SPST-NO, 0.05A, 12V, -> B3U-1000P SWITCH, SPST-NO, 0.05A, 12V, SMD; Manufacturer Omron Electronics Inc-EMC Div -> OMRON ELECTRONIC COMPONENTS; Vendor Digi-Key -> Farnell; Vendor Part Number SW1020CT-ND -> 1333652
Connections:
- net +1V2: now also C16.1, C18.1, C20.1, C22.1
- net +3V3: now also C14.1, C15.1, C17.1, C19.1, C21.1, C23.1; no longer U1.46 (VCCIO_2), U1.57 (VCCIO_2)
- net DIQ1_D0: now also U1.79 (IOR_53_115); no longer U1.73 (IOR_48_109)
- net DIQ1_D1: now also U1.73 (IOR_48_109); no longer U1.74 (IOR_49_110)
- net DIQ1_D11: now also U1.134 (IOT_87_212); no longer U1.91 (IOR_59_139)
- net DIQ1_D2: now also U1.80 (IOR_54_116); no longer U1.75 (IOR_50_111)
- net DIQ1_D3: now also U1.74 (IOR_49_110); no longer U1.76 (IOR_51_112)
- net DIQ1_D4: now also U1.81 (IOR_55_117); no longer U1.78 (IOR_52_114)
- net DIQ1_D5: now also U1.75 (IOR_50_111); no longer U1.79 (IOR_53_115)
- net DIQ1_D6: now also U1.87 (IOR_56_136); no longer U1.80 (IOR_54_116)
- net DIQ1_D7: now also U1.76 (IOR_51_112); no longer U1.81 (IOR_55_117)
- net DIQ1_D8: now also U1.88 (IOR_57_137); no longer U1.87 (IOR_56_136)
- net DIQ1_D9: now also U1.91 (IOR_59_139); no longer U1.88 (IOR_57_137)
- net DIQ1_SEL: now also U1.78 (IOR_52_114); no longer U1.114 (IOT_75_171)
- net DIQ2_D1: now also U1.129 (IOT_85_198); no longer U1.95 (IOR_62_144)
- net DIQ2_D10: now also U1.99 (IOR_66_152); no longer U1.106 (IOR_71_166)
- net DIQ2_D11: now also U1.119 (IOT_80_178); no longer U1.107 (IOR_72_167)
- net DIQ2_D2: now also U1.95 (IOR_62_144); no longer U1.96 (IOR_63_146)
- net DIQ2_D3: now also U1.128 (IOT_84_197); no longer U1.97 (IOR_64_147)
- net DIQ2_D4: now also U1.96 (IOR_63_146); no longer U1.98 (IOR_65_148)
- net DIQ2_D5: now also U1.122 (IOT_83_190); no longer U1.99 (IOR_66_152)
- net DIQ2_D6: now also U1.97 (IOR_64_147); no longer U1.101 (IOR_67_160)
- net DIQ2_D7: now also U1.121 (IOT_82_181); no longer U1.102 (IOR_68_161)
- net DIQ2_D8: now also U1.98 (IOR_65_148); no longer U1.104 (IOR_69_164)
- net DIQ2_D9: now also U1.120 (IOT_81_179); no longer U1.105 (IOR_70_165)
- net DIQ2_SEL: now also U1.93 (IOR_60_140); no longer U1.115 (IOT_76_172)
- net FCLK1: now also U1.118 (IOT_79_177); no longer U1.116 (IOT_77_173)
- net FCLK2: now also U1.101 (IOR_67_160); no longer U1.117 (IOT_78_174)
- net GND: now also SW1.1 (Base), C14.2, C15.2, C16.2, C17.2, C18.2, C19.2, C20.2, C21.2, C22.2, C23.2
- net ICE_CRESET_B: now also SW1.2 (Coll)
- net RFDIO_GPIO0: now also U1.102 (IOR_68_161); no longer U1.119 (IOT_80_178)
- net RFDIO_GPIO1: now also U1.104 (IOR_69_164); no longer U1.120 (IOT_81_179)
- net RFDIO_GPIO2: now also U1.105 (IOR_70_165); no longer U1.121 (IOT_82_181)
- net RFDIO_REF_CLK_IN: now also U1.106 (IOR_71_166); no longer U1.135 (IOT_88_213)
- net RFDIO_RESET: now also U1.117 (IOT_78_174); no longer U1.118 (IOT_79_177)
- net RFDIO_SPI_CLK: now also U1.114 (IOT_75_171); no longer U1.129 (IOT_85_198)
- net RFDIO_SPI_EN: now also U1.113 (IOT_74_170); no longer U1.134 (IOT_87_212)
- net RFDIO_SPI_MISO: now also U1.115 (IOT_76_172); no longer U1.128 (IOT_84_197)
- net RFDIO_SPI_MOSI: now also U1.116 (IOT_77_173); no longer U1.122 (IOT_83_190)
- net TXEN: now also U1.107 (IOR_72_167); no longer U1.113 (IOT_74_170)
- no-connect marks 0 -> 34
Other:
- note added: "Filter"
- note added: "Place near to Pins"
- moved on the sheet: C1, C10, C11, C12, C13, C2, C6, C7, C8, C9, R12, R7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
