File: board/KiCad/ice40.sch (KiCad schematic (older format))
At the start: 34 parts, among them SW1 ICE_RESET, U1 iCE40_1K4K_TQ144

Commit message: Improve design
* PMOS on input voltage for polarity
* Re-design board to add mount holes and better routing
Connections:
- net DIQ1_D0: now also U1.74 (IOR_49_110); no longer U1.79 (IOR_53_115)
- net DIQ1_D1: now also U1.78 (IOR_52_114); no longer U1.73 (IOR_48_109)
- net DIQ1_D11: now also U1.93 (IOR_60_140); no longer U1.134 (IOT_87_212)
- net DIQ1_D2: now also U1.75 (IOR_50_111); no longer U1.80 (IOR_54_116)
- net DIQ1_D3: now also U1.79 (IOR_53_115); no longer U1.74 (IOR_49_110)
- net DIQ1_D4: now also U1.76 (IOR_51_112); no longer U1.81 (IOR_55_117)
- net DIQ1_D5: now also U1.80 (IOR_54_116); no longer U1.75 (IOR_50_111)
- net DIQ1_D7: now also U1.81 (IOR_55_117); no longer U1.76 (IOR_51_112)
- net DIQ1_SEL: now also U1.73 (IOR_48_109); no longer U1.78 (IOR_52_114)
- net DIQ2_D0: now also U1.97 (IOR_64_147); no longer U1.94 (IOR_61_141)
- net DIQ2_D1: now also U1.94 (IOR_61_141); no longer U1.129 (IOT_85_198)
- net DIQ2_D10: now also U1.107 (IOR_72_167); no longer U1.99 (IOR_66_152)
- net DIQ2_D11: now also U1.113 (IOT_74_170); no longer U1.119 (IOT_80_178)
- net DIQ2_D2: now also U1.99 (IOR_66_152); no longer U1.95 (IOR_62_144)
- net DIQ2_D3: now also U1.95 (IOR_62_144); no longer U1.128 (IOT_84_197)
- net DIQ2_D4: now also U1.101 (IOR_67_160); no longer U1.96 (IOR_63_146)
- net DIQ2_D5: now also U1.98 (IOR_65_148); no longer U1.122 (IOT_83_190)
- net DIQ2_D6: now also U1.105 (IOR_70_165); no longer U1.97 (IOR_64_147)
- net DIQ2_D7: now also U1.102 (IOR_68_161); no longer U1.121 (IOT_82_181)
- net DIQ2_D8: now also U1.106 (IOR_71_166); no longer U1.98 (IOR_65_148)
- net DIQ2_D9: now also U1.104 (IOR_69_164); no longer U1.120 (IOT_81_179)
- net DIQ2_SEL: now also U1.96 (IOR_63_146); no longer U1.93 (IOR_60_140)
- net FCLK1: now also U1.114 (IOT_75_171); no longer U1.118 (IOT_79_177)
- net FCLK2: now also U1.112 (IOT_73_169); no longer U1.101 (IOR_67_160)
- net PIO10: now also U1.9 (IOL_4A_5A); no longer U1.8 (IOL_3B_4B)
- net PIO12: now also U1.3 (IOL_2A_3A); no longer U1.1 (IOL_1A_2A)
- net PIO13: now also U1.2 (IOL_1B_2B); no longer U1.3 (IOL_2A_3A)
- net PIO14: now also U1.1 (IOL_1A_2A); no longer U1.7 (IOL_3A_4A)
- net PIO15: now also U1.4 (IOL_2B_3B); no longer U1.9 (IOL_4A_5A)
- net PIO8: now also U1.7 (IOL_3A_4A); no longer U1.2 (IOL_1B_2B)
- net PIO9: now also U1.8 (IOL_3B_4B); no longer U1.4 (IOL_2B_3B)
- net RFDIO_GPIO0: now also U1.118 (IOT_79_177); no longer U1.102 (IOR_68_161)
- net RFDIO_GPIO1: now also U1.119 (IOT_80_178); no longer U1.104 (IOR_69_164)
- net RFDIO_GPIO2: now also U1.120 (IOT_81_179); no longer U1.105 (IOR_70_165)
- net RFDIO_REF_CLK_IN: now also U1.121 (IOT_82_181); no longer U1.106 (IOR_71_166)
- net RFDIO_RESET: now also U1.115 (IOT_76_172); no longer U1.117 (IOT_78_174)
- net RFDIO_SPI_CLK: now also U1.128 (IOT_84_197); no longer U1.114 (IOT_75_171)
- net RFDIO_SPI_EN: now also U1.129 (IOT_85_198); no longer U1.113 (IOT_74_170)
- net RFDIO_SPI_MISO: now also U1.117 (IOT_78_174); no longer U1.115 (IOT_76_172)
- net RXEN: now also U1.134 (IOT_87_212); no longer U1.112 (IOT_73_169)
- net TXEN: now also U1.122 (IOT_83_190); no longer U1.107 (IOR_72_167)
Changed lines of the file:
@@
 	1    0    0    -1
 $EndComp
-Text GLabel 8600 900  2    60   Input ~ 0
+Text GLabel 8600 1100 2    60   Input ~ 0
 PIO12
+Text GLabel 8600 1300 2    60   Input ~ 0
+PIO8
 Text GLabel 8950 1000 2    60   Input ~ 0
-PIO8
-Text GLabel 8600 1100 2    60   Input ~ 0
 PIO13
-Text GLabel 8950 1200 2    60   Input ~ 0
+Text GLabel 8950 1400 2    60   Input ~ 0
 PIO9
-Text GLabel 8950 1400 2    60   Input ~ 0
+Text GLabel 8600 1500 2    60   Input ~ 0
 PIO10
 Text GLabel 8950 1600 2    60   Input ~ 0
 PIO11
-Text GLabel 8600 1300 2    60   Input ~ 0
+Text GLabel 8600 900  2    60   Input ~ 0
 PIO14
-Text GLabel 8600 1500 2    60   Input ~ 0
+Text GLabel 8950 1200 2    60   Input ~ 0
 PIO15
 Text GLabel 8600 1700 2    60   Input ~ 0
@@
 3V3_PMOD
 $Comp
-L +3V3 #PWR35
+L +3V3 #PWR24
 U 1 1 56ABB1F6
 P 9650 6000
-F 0 "#PWR35" H 9650 5850 50  0001 C CNN
+F 0 "#PWR24" H 9650 5850 50  0001 C CNN
 F 1 "+3V3" H 9668 6174 50  0000 C CNN
 F 2 "" H 9650 6000 50  0000 C CNN
@@
 1V2_LDO
 $Comp
-L +1V2 #PWR36
+L +1V2 #PWR25
 U 1 1 56ABBB92
 P 9850 6250
-F 0 "#PWR36" H 9850 6100 50  0001 C CNN
+F 0 "#PWR25" H 9850 6100 50  0001 C CNN
 F 1 "+1V2" H 9850 6390 50  0000 C CNN
 F 2 "" H 9850 6250 60  0000 C CNN
@@
 $EndComp
 $Comp
-L +1V2 #PWR6
+L +1V2 #PWR8
 U 1 1 56ABC35C
 P 2300 2650
-F 0 "#PWR6" H 2300 2500 50  0001 C CNN
+F 0 "#PWR8" H 2300 2500 50  0001 C CNN
 F 1 "+1V2" H 2300 2790 50  0000 C CNN
 F 2 "" H 2300 2650 60  0000 C CNN
@@
 $EndComp
 $Comp
-L +1V2 #PWR9
+L +1V2 #PWR11
 U 1 1 56ABC562
 P 3450 3700
-F 0 "#PWR9" H 3450 3550 50  0001 C CNN
+F 0 "#PWR11" H 3450 3550 50  0001 C CNN
 F 1 "+1V2" H 3450 3840 50  0000 C CNN
 F 2 "" H 3450 3700 60  0000 C CNN
@@
 $EndComp
 $Comp
-L +3V3 #PWR1
+L +3V3 #PWR5
 U 1 1 56ABE3D7
 P 2000 2975
-F 0 "#PWR1" H 2000 2825 50  0001 C CNN
+F 0 "#PWR5" H 2000 2825 50  0001 C CNN
 F 1 "+3V3" H 2018 3149 50  0000 C CNN
 F 2 "" H 2000 2975 50  0000 C CNN
@@
 $EndComp
 $Comp
-L GND #PWR4
+L GND #PWR6
 U 1 1 56ABE688
 P 2250 1350
-F 0 "#PWR4" H 2250 1100 50  0001 C CNN
+F 0 "#PWR6" H 2250 1100 50  0001 C CNN
 F 1 "GND" H 2250 1200 50  0000 C CNN
 F 2 "" H 2250 1350 60  0000 C CNN
@@
 	1    0    0    -1
 $EndComp
-Text GLabel 5200 1450 2    60   Input ~ 0
+Text GLabel 5200 1050 2    60   Input ~ 0
 DIQ1_D0
+Text GLabel 2050 6100 2    60   Input ~ 0
+RXEN
+Text GLabel 2050 5800 2    60   Input ~ 0
+TXEN
+Text GLabel 5200 950  2    60   Input ~ 0
+DIQ1_SEL
+Text GLabel 5200 2450 2    60   Input ~ 0
+DIQ2_SEL
+Text GLabel 2050 5000 2    60   Input ~ 0
+FCLK1
 Text GLabel 2050 4800 2    60   Input ~ 0
-RXEN
-Text GLabel 5200 3350 2    60   Input ~ 0
-TXEN
-Text GLabel 5200 1350 2    60   Input ~ 0
-DIQ1_SEL
-Text GLabel 5200 2150 2    60   Input ~ 0
-DIQ2_SEL
-Text GLabel 2050 5400 2    60   Input ~ 0
-FCLK1
-Text GLabel 5200 2850 2    60   Input ~ 0
 FCLK2
 Text GLabel 1950 1150 2    60   Input ~ 0
 ICE_CLK_IN
-Text GLabel 2050 5300 2    60   Input ~ 0
+Text GLabel 2050 5100 2    60   Input ~ 0
 RFDIO_RESET
-Text GLabel 5200 2950 2    60   Input ~ 0
+Text GLabel 2050 5400 2    60   Input ~ 0
 RFDIO_GPIO0
-Text GLabel 5200 3050 2    60   Input ~ 0
+Text GLabel 2050 5500 2    60   Input ~ 0
 RFDIO_GPIO1
-Text GLabel 5200 3150 2    60   Input ~ 0
+Text GLabel 2050 5600 2    60   Input ~ 0
 RFDIO_GPIO2
 Text GLabel 2050 5200 2    60   Input ~ 0
 RFDIO_SPI_MOSI
-Text GLabel 2050 5100 2    60   Input ~ 0
+Text GLabel 2050 5300 2    60   Input ~ 0
 RFDIO_SPI_MISO
-Text GLabel 2050 5000 2    60   Input ~ 0
+Text GLabel 2050 5900 2    60   Input ~ 0
 RFDIO_SPI_CLK
-Text GLabel 2050 4900 2    60   Input ~ 0
+Text GLabel 2050 6000 2    60   Input ~ 0
 RFDIO_SPI_EN
-Text GLabel 5200 3250 2    60   Input ~ 0
+Text GLabel 2050 5700 2    60   Input ~ 0
 RFDIO_REF_CLK_IN
 Text GLabel 1700 1050 2    60   Input ~ 0
@@
 ICE_SS
 $Comp
-L +3V3 #PWR5
+L +3V3 #PWR7
 U 1 1 56BB434D
 P 2250 4100
-F 0 "#PWR5" H 2250 3950 50  0001 C CNN
+F 0 "#PWR7" H 2250 3950 50  0001 C CNN
 F 1 "+3V3" H 2268 4274 50  0000 C CNN
 F 2 "" H 2250 4100 50  0000 C CNN
@@
 $EndComp
 $Comp
-L +3V3 #PWR31
+L +3V3 #PWR20
 U 1 1 56BB5247
 P 7650 3800
-F 0 "#PWR31" H 7650 3650 50  0001 C CNN
+F 0 "#PWR20" H 7650 3650 50  0001 C CNN
 F 1 "+3V3" H 7668 3974 50  0000 C CNN
 F 2 "" H 7650 3800 50  0000 C CNN
@@
 $EndComp
 $Comp
-L +3V3 #PWR33
+L +3V3 #PWR22
 U 1 1 56BB576D
 P 9225 3750
-F 0 "#PWR33" H 9225 3600 50  0001 C CNN
+F 0 "#PWR22" H 9225 3600 50  0001 C CNN
 F 1 "+3V3" H 9243 3924 50  0000 C CNN
 F 2 "" H 9225 3750 50  0000 C CNN
@@
 $EndComp
 $Comp
-L GND #PWR34
+L GND #PWR23
 U 1 1 56BB5D2F
 P 9225 5050
-F 0 "#PWR34" H 9225 4800 50  0001 C CNN
+F 0 "#PWR23" H 9225 4800 50  0001 C CNN
 F 1 "GND" H 9225 4900 50  0000 C CNN
 F 2 "" H 9225 5050 60  0000 C CNN
@@
 $EndComp
 $Comp
-L GND #PWR17
+L GND #PWR15
 U 1 1 56BB9E95
 P 4750 4875
-F 0 "#PWR17" H 4750 4625 50  0001 C CNN
+F 0 "#PWR15" H 4750 4625 50  0001 C CNN
 F 1 "GND" H 4750 4725 50  0000 C CNN
 F 2 "" H 4750 4875 60  0000 C CNN
@@
 $EndComp
 $Comp
-L +3V3 #PWR16
+L +3V3 #PWR14
 U 1 1 56BB9ED0
 P 4750 4325
-F 0 "#PWR16" H 4750 4175 50  0001 C CNN
+F 0 "#PWR14" H 4750 4175 50  0001 C CNN
 F 1 "+3V3" H 4768 4499 50  0000 C CNN
 F 2 "" H 4750 4325 50  0000 C CNN
@@
 $EndComp
 $Comp
-L GND #PWR19
+L GND #PWR17
 U 1 1 56BBA5A4
 P 5125 5650
-F 0 "#PWR19" H 5125 5400 50  0001 C CNN
+F 0 "#PWR17" H 5125 5400 50  0001 C CNN
 F 1 "GND" H 5125 5500 50  0000 C CNN
 F 2 "" H 5125 5650 60  0000 C CNN
@@
 $EndComp
 $Comp
-L +1V2 #PWR18
+L +1V2 #PWR16
 U 1 1 56BBA638
 P 5125 5100
-F 0 "#PWR18" H 5125 4950 50  0001 C CNN
+F 0 "#PWR16" H 5125 4950 50  0001 C CNN
 F 1 "+1V2" H 5125 5240 50  0000 C CNN
 F 2 "" H 5125 5100 60  0000 C CNN
@@
 $EndComp
 $Comp
-L GND #PWR32
+L GND #PWR21
 U 1 1 56BD2668
 P 7650 5400
-F 0 "#PWR32" H 7650 5150 50  0001 C CNN
+F 0 "#PWR21" H 7650 5150 50  0001 C CNN
 F 1 "GND" H 7650 5250 50  0000 C CNN
 F 2 "" H 7650 5400 60  0000 C CNN
@@
 $EndComp
 $Comp
-L +3V3 #PWR7
+L +3V3 #PWR9
 U 1 1 56BE4EE6
 P 2400 4250
-F 0 "#PWR7" H 2400 4100 50  0001 C CNN
+F 0 "#PWR9" H 2400 4100 50  0001 C CNN
 F 1 "+3V3" H 2418 4424 50  0000 C CNN
 F 2 "" H 2400 4250 50  0000 C CNN
@@
 $EndComp
 $Comp
-L GND #PWR8
+L GND #PWR10
 U 1 1 56BE5949
 P 2850 7150
-F 0 "#PWR8" H 2850 6900 50  0001 C CNN
+F 0 "#PWR10" H 2850 6900 50  0001 C CNN
 F 1 "GND" H 2850 7000 50  0000 C CNN
 F 2 "" H 2850 7150 60  0000 C CNN
@@
 Text Notes 8275 5300 0    60   ~ 0
 ICE reset
-Text GLabel 5200 950  2    60   Input ~ 0
+Text GLabel 5200 1350 2    60   Input ~ 0
 DIQ1_D1
+Text GLabel 5200 1150 2    60   Input ~ 0
+DIQ1_D2
+Text GLabel 5200 1450 2    60   Input ~ 0
+DIQ1_D3
+Text GLabel 5200 1250 2    60   Input ~ 0
+DIQ1_D4
 Text GLabel 5200 1550 2    60   Input ~ 0
-DIQ1_D2
-Text GLabel 5200 1050 2    60   Input ~ 0
-DIQ1_D3
-Text GLabel 5200 1650 2    60   Input ~ 0
-DIQ1_D4
-Text GLabel 5200 1150 2    60   Input ~ 0
 DIQ1_D5
 Text GLabel 5200 1750 2    60   Input ~ 0
 DIQ1_D6
-Text GLabel 5200 1250 2    60   Input ~ 0
+Text GLabel 5200 1650 2    60   Input ~ 0
 DIQ1_D7
 Text GLabel 5200 1850 2    60   Input ~ 0
@@
 Text GLabel 5200 1950 2    60   Input ~ 0
 DIQ1_D10
-Text GLabel 2050 6100 2    60   Input ~ 0
+Text GLabel 5200 2150 2    60   Input ~ 0
 DIQ1_D11
+Text GLabel 5200 2550 2    60   Input ~ 0
+DIQ2_D0
+Text GLabel 5200 2750 2    60   Input ~ 0
+DIQ2_D2
+Text GLabel 5200 2850 2    60   Input ~ 0
+DIQ2_D4
+Text GLabel 5200 3150 2    60   Input ~ 0
+DIQ2_D6
+Text GLabel 5200 3250 2    60   Input ~ 0
+DIQ2_D8
+Text GLabel 5200 3350 2    60   Input ~ 0
+DIQ2_D10
 Text GLabel 5200 2250 2    60   Input ~ 0
-DIQ2_D0
+DIQ2_D1
 Text GLabel 5200 2350 2    60   Input ~ 0
-DIQ2_D2
-Text GLabel 5200 2450 2    60   Input ~ 0
-DIQ2_D4
-Text GLabel 5200 2550 2    60   Input ~ 0
-DIQ2_D6
+DIQ2_D3
 Text GLabel 5200 2650 2    60   Input ~ 0
-DIQ2_D8
-Text GLabel 5200 2750 2    60   Input ~ 0
-DIQ2_D10
-Text GLabel 2050 6000 2    60   Input ~ 0
-DIQ2_D1
-Text GLabel 2050 5900 2    60   Input ~ 0
-DIQ2_D3
-Text GLabel 2050 5800 2    60   Input ~ 0
 DIQ2_D5
-Text GLabel 2050 5700 2    60   Input ~ 0
+Text GLabel 5200 2950 2    60   Input ~ 0
 DIQ2_D7
-Text GLabel 2050 5600 2    60   Input ~ 0
+Text GLabel 5200 3050 2    60   Input ~ 0
 DIQ2_D9
-Text GLabel 2050 5500 2    60   Input ~ 0
+Text GLabel 2050 4900 2    60   Input ~ 0
 DIQ2_D11
 NoConn ~ 1700 6700
@@
 Connection ~ 5525 7225
 $Comp
-L GND #PWR11
+L GND #PWR13
 U 1 1 56C2D636
 P 3525 6600
-F 0 "#PWR11" H 3525 6350 50  0001 C CNN
+F 0 "#PWR13" H 3525 6350 50  0001 C CNN
 F 1 "GND" H 3533 6426 50  0000 C CNN
 F 2 "" H 3525 6600 50  0000 C CNN
@@
 $EndComp
 $Comp
-L GND #PWR21
+L GND #PWR19
 U 1 1 56C2D6BD
 P 5200 7250
-F 0 "#PWR21" H 5200 7000 50  0001 C CNN
+F 0 "#PWR19" H 5200 7000 50  0001 C CNN
 F 1 "GND" H 5208 7076 50  0000 C CNN
 F 2 "" H 5200 7250 50  0000 C CNN
@@
 $EndComp
 $Comp
-L +3V3 #PWR10
+L +3V3 #PWR12
 U 1 1 56C2D827
 P 3525 6250
-F 0 "#PWR10" H 3525 6100 50  0001 C CNN
+F 0 "#PWR12" H 3525 6100 50  0001 C CNN
 F 1 "+3V3" H 3543 6424 50  0000 C CNN
 F 2 "" H 3525 6250 50  0000 C CNN
@@
 $EndComp
 $Comp
-L +1V2 #PWR20
+L +1V2 #PWR18
 U 1 1 56C2D8A7
 P 5200 6950
-F 0 "#PWR20" H 5200 6800 50  0001 C CNN
+F 0 "#PWR18" H 5200 6800 50  0001 C CNN
 F 1 "+1V2" H 5200 7090 50  0000 C CNN
 F 2 "" H 5200 6950 60  0000 C CNN

Commit message: Housekeeping
Structure libraries and put proper licenses to them.
Parts:
- D2: footprint pmod:SOD-123_Handsoldering -> lms6002-pmod:SOD-123_Handsoldering
- SW1: footprint pmod:B3U-1000P_Handsoldering -> lms6002-pmod:B3U-1000P_Handsoldering
Changed lines of the file:
@@
 LIBS:contrib
 LIBS:valves
+LIBS:lms6002-pmod
 LIBS:ice40_1k4k_tq144
 LIBS:myriad
-LIBS:pmod
-LIBS:LMS6002-Pmod-cache
 EELAYER 25 0
 EELAYER END
@@
 F 0 "D2" H 2050 4380 50  0000 L CNN
 F 1 "Schottky 0520" H 1820 4220 50  0000 L CNN
-F 2 "pmod:SOD-123_Handsoldering" V 2100 4300 60  0001 C CNN
+F 2 "lms6002-pmod:SOD-123_Handsoldering" V 2100 4300 60  0001 C CNN
 F 3 "" V 2100 4300 60  0000 C CNN
 	1    2100 4300
@@
 F 0 "SW1" H 9225 4725 60  0000 C CNN
 F 1 "ICE_RESET" H 9250 4850 60  0001 C CNN
-F 2 "pmod:B3U-1000P_Handsoldering" H 9275 4975 60  0001 C CNN
+F 2 "lms6002-pmod:B3U-1000P_Handsoldering" H 9275 4975 60  0001 C CNN
 F 3 "" H 9225 4625 60  0000 C CNN
 F 4 "B3U-1000P" H 9250 5175 60  0001 C CNN "Manufacturer Part Number"
