File: board/KiCad/Pmod.sch (KiCad schematic (older format))
At the start: 2 parts, among them P1 PMOD_2x6, P2 PMOD_2x6

Commit message: Housekeeping
Structure libraries and put proper licenses to them.
Parts:
- P1: footprint pmod:Pmod -> lms6002-pmod:Pmod
- P2: footprint pmod:Pmod -> lms6002-pmod:Pmod_no_header
Changed lines of the file:
@@
 LIBS:contrib
 LIBS:valves
+LIBS:lms6002-pmod
 LIBS:ice40_1k4k_tq144
 LIBS:myriad
-LIBS:pmod
-LIBS:LMS6002-Pmod-cache
 EELAYER 25 0
 EELAYER END
@@
 F 0 "P1" H 5000 4216 50  0000 C CNN
 F 1 "PMOD_2x6" H 5000 4124 50  0000 C CNN
-F 2 "pmod:Pmod" H 5000 2550 50  0001 C CNN
+F 2 "lms6002-pmod:Pmod" H 5000 2550 50  0001 C CNN
 F 3 "" H 5000 2550 50  0000 C CNN
 	1    5000 3750
@@
 F 0 "P2" H 6800 4216 50  0000 C CNN
 F 1 "PMOD_2x6" H 6800 4124 50  0000 C CNN
-F 2 "pmod:Pmod" H 6800 2550 50  0001 C CNN
+F 2 "lms6002-pmod:Pmod_no_header" H 6800 2550 50  0001 C CNN
 F 3 "" H 6800 2550 50  0000 C CNN
 	1    6800 3750
