File: board/KiCad/power_supply.sch (KiCad schematic (older format))
At the start: 12 parts, among them CON1 BARREL_JACK, J3 SELECT_DIV, Q1 Q_PMOS_GSD, U2 LD6815, U3 LTC1799

Commit message: Housekeeping
Structure libraries and put proper licenses to them.
Parts:
- CON1: footprint Connect:BARREL_JACK -> lms6002-pmod:BARREL_JACK
- D1: footprint pmod:SOD-123F_Handsoldering -> lms6002-pmod:SOD-123F_Handsoldering
- U2: footprint pmod:SOT-753_(TSOP-5)_Handsoldering -> lms6002-pmod:SOT-753_(TSOP-5)_Handsoldering
- U3: footprint pmod:TSOT-23_Handsoldering -> lms6002-pmod:TSOT-23_Handsoldering
Changed lines of the file:
@@
 LIBS:contrib
 LIBS:valves
+LIBS:lms6002-pmod
 LIBS:ice40_1k4k_tq144
 LIBS:myriad
-LIBS:pmod
-LIBS:LMS6002-Pmod-cache
 EELAYER 25 0
 EELAYER END
@@
 F 0 "CON1" H 2100 2050 60  0000 C CNN
 F 1 "BARREL_JACK" H 2100 1600 60  0000 C CNN
-F 2 "Connect:BARREL_JACK" H 2100 1800 60  0001 C CNN
+F 2 "lms6002-pmod:BARREL_JACK" H 2100 1800 60  0001 C CNN
 F 3 "" H 2100 1800 60  0000 C CNN
 	1    2100 1800
@@
 F 0 "U2" H 6550 2750 60  0000 C CNN
 F 1 "LD6815" H 6550 2900 60  0000 C CNN
-F 2 "pmod:SOT-753_(TSOP-5)_Handsoldering" H 6550 2750 60  0001 C CNN
+F 2 "lms6002-pmod:SOT-753_(TSOP-5)_Handsoldering" H 6550 2750 60  0001 C CNN
 F 3 "" H 6550 2750 60  0000 C CNN
 	1    6550 2750
@@
 F 0 "D1" H 4600 2200 50  0000 C CNN
 F 1 "5V-SOD-123F" H 4600 2000 50  0000 C CNN
-F 2 "pmod:SOD-123F_Handsoldering" H 4600 2100 50  0001 C CNN
+F 2 "lms6002-pmod:SOD-123F_Handsoldering" H 4600 2100 50  0001 C CNN
 F 3 "" H 4600 2100 50  0000 C CNN
 	1    4600 2100
@@
 F 0 "U3" H 3450 6100 60  0000 C CNN
 F 1 "LTC1799" H 3450 7100 60  0000 C CNN
-F 2 "pmod:TSOT-23_Handsoldering" H 3450 6100 60  0001 C CNN
+F 2 "lms6002-pmod:TSOT-23_Handsoldering" H 3450 6100 60  0001 C CNN
 F 3 "" H 3450 6100 60  0000 C CNN
 	1    3450 6100
